Commit message: 4

File: src/my_r2d2/urdf/r2d2.urdf (robot description, URDF)
Before this commit: robot macroed, 6 links, 5 joints
Links:
- removed link lens
- added link eye
- added link lense; collision cylinder length=${lenslen} radius=${lensrad}; visual cylinder length=${lenslen} radius=${lensrad}
Joints:
- removed joint head_lens
- added joint head_lense: type fixed, parent box, child eye
- added joint lense_eye: type fixed, parent eye, child lense, origin xyz=0 0 0 rpy=${pi/2} ${pi} ${pi/2}
